File: dc-motor-driver.kicad_sch (KiCad schematic)
At the start: 12 parts, among them U2 DRV8874

Commit message: schem: add second dc motor driver
Parts:
- renumbered C8 to C6, C9 to C7, C6 to C8, C7 to C9, JP2 to JP1, JP1 to JP2, R6 to R4, R7 to R5, R5 to R6, R4 to R7

Commit message: schem: add various test points
Parts:
- added TP4: TestPoint, TestPoint:TestPoint_Pad_D2.0mm, symbol Connector:TestPoint
Connections:
- net IPROPI: now also TP4.1
Changed lines of the file:
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@@
+	)
+	(junction
+		(at 130.81 104.14)
+		(diameter 0)
+		(color 0 0 0 0)
 	)
 	(junction
@@
 	(wire
 		(pts
-			(xy 123.19 104.14) (xy 133.35 104.14)
+			(xy 123.19 104.14) (xy 130.81 104.14)
 		)
 		(stroke
@@
 		(pts
 			(xy 172.72 107.95) (xy 172.72 106.68)
+		)
+		(stroke
+			(width 0)
+			(type default)
+		)
+	)
+	(wire
+		(pts
+			(xy 130.81 104.14) (xy 133.35 104.14)
 		)
 		(stroke
@@
 		(on_board yes)
 		(dnp no)
-		(fields_autoplaced yes)
 		(property "Reference" "R6"
-			(at 125.73 107.9499 0)
+			(at 125.222 107.95 0)
 			(effects
 				(font
@@
 		)
 		(property "Value" "1k"
-			(at 125.73 110.4899 0)
+			(at 125.222 110.49 0)
 			(effects
 				(font
@@
 					(unit 1)
 				)
+			)
+		)
+	)
+	(symbol
+		(lib_id "Connector:TestPoint")
+		(at 130.81 104.14 180)
+		(unit 1)
+		(exclude_from_sim no)
+		(in_bom no)
+		(on_board yes)
+		(dnp no)
+		(property "Reference" "TP4"
+			(at 132.842 109.474 0)
+			(effects
+				(font
+					(size 1.27 1.27)
+				)
+				(justify left)
+			)
+		)
+		(property "Value" "TestPoint"
+			(at 128.27 106.1721 0)
+			(effects
+				(font
+					(size 1.27 1.27)
+				)
+				(justify left)
+				(hide yes)
+			)
+		)
+		(property "Footprint" "TestPoint:TestPoint_Pad_D2.0mm"
+			(at 125.73 104.14 0)
+			(effects
+				(font
+					(size 1.27 1.27)
+				)
+				(hide yes)
+			)
+		)
+		(property "Datasheet" "~"
+			(at 125.73 104.14 0)
+			(effects
+				(font
+					(size 1.27 1.27)
+				)
+				(hide yes)
+			)
+		)
+		(property "Description" "test point"
+			(at 130.81 104.14 0)
+			(effects
+				(font
+					(size 1.27 1.27)
+				)
+				(hide yes)
+			)
+		)
+		(pin "1"
+		)
+		(instances
+			(project "valrob-carte-moteur-cdf-1"
+				(path "/b89f538c-def5-4450-bb35-40e96c574400/046dd584-44f1-462d-a721-c6fc6e1dad4e"
+					(reference "TP4")
+					(unit 1)
+				)
+				(path "/b89f538c-def5-4450-bb35-40e96c574400/4610ebb9-9c7e-4d93-9787-ad1280502022"
+					(reference "TP5")
+					(unit 1)
+				)

Commit message: schem: reannotate
Parts:
- renumbered C8 to C10, C9 to C11, C6 to C8, C7 to C9, R4 to R10, R5 to R11, R6 to R12, R7 to R13, R8 to R14, TP4 to TP5, U2 to U4

Commit message: schem: add sheet titles
Other:
- company: (none) -> Valrobotik
- title: (none) -> Carte moteur CDF 1
Changed lines of the file:
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@@
 	(generator_version "9.0")
 	(paper "A4")
+	(title_block
+		(title "Carte moteur CDF 1")
+		(date "2025-11-23")
+		(rev "01")
+		(company "Valrobotik")
+		(comment 1 "5A DC motor driver")
+	)
 	(junction
 		(at 151.13 114.3)

Commit message: schem: add components footprints
Parts:
- C10, C8, C9: footprint (none) -> Capacitor_SMD:C_0603_1608Metric
- C11: footprint (none) -> Capacitor_SMD:CP_Elec_6.3x7.7
- JP1, JP2: footprint (none) -> Connector_PinHeader_2.54mm:PinHeader_1x03_P2.54mm_Vertical
- R10, R11, R12, R14: footprint (none) -> Resistor_SMD:R_0603_1608Metric
Changed lines of the file:
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@@
 			)
 		)
-		(property "Footprint" ""
+		(property "Footprint" "Resistor_SMD:R_0603_1608Metric"
 			(at 121.412 109.22 90)
 			(effects
@@
 			)
 		)
-		(property "Footprint" ""
+		(property "Footprint" "Connector_PinHeader_2.54mm:PinHeader_1x03_P2.54mm_Vertical"
 			(at 134.62 114.3 0)
 			(effects
@@
 			)
 		)
-		(property "Footprint" ""
+		(property "Footprint" "Resistor_SMD:R_0603_1608Metric"
 			(at 146.05 112.522 90)
 			(effects
@@
 			)
 		)
-		(property "Footprint" ""
+		(property "Footprint" "Resistor_SMD:R_0603_1608Metric"
 			(at 116.332 93.98 90)
 			(effects
@@
 			)
 		)
-		(property "Footprint" ""
+		(property "Footprint" "Capacitor_SMD:C_0603_1608Metric"
 			(at 168.91 96.52 0)
 			(effects
@@
 			)
 		)
-		(property "Footprint" ""
+		(property "Footprint" "Capacitor_SMD:CP_Elec_6.3x7.7"
 			(at 179.3748 115.57 0)
 			(effects
@@
 			)
 		)
-		(property "Footprint" ""
+		(property "Footprint" "Capacitor_SMD:C_0603_1608Metric"
 			(at 168.91 104.14 0)
 			(effects
@@
 			)
 		)
-		(property "Footprint" ""
+		(property "Footprint" "Capacitor_SMD:C_0603_1608Metric"
 			(at 171.7548 115.57 0)
 			(effects
@@
 			)
 		)
-		(property "Footprint" ""
+		(property "Footprint" "Connector_PinHeader_2.54mm:PinHeader_1x03_P2.54mm_Vertical"
 			(at 177.8 93.98 0)
 			(effects
@@
 			)
 		)
-		(property "Footprint" ""
+		(property "Footprint" "Resistor_SMD:R_0603_1608Metric"
 			(at 116.332 104.14 90)
 			(effects

Commit message: schem: add ordering info to BOM
Parts:
- C10, C9: Basic (none) -> Y; JLCPCB Part # (none) -> C14663; Manufacturer (none) -> YAGEO; Manufacturer Part Number (none) -> CC0603KRX7R9BB104
- C11: Basic (none) -> X; JLCPCB Part # (none) -> C2918361; Manufacturer (none) -> ROQANG; Manufacturer Part Number (none) -> RVT1E221M0607
- C8: Basic (none) -> Y; JLCPCB Part # (none) -> C21122; Manufacturer (none) -> Samsung Electro-Mechanics; Manufacturer Part Number (none) -> CL10B223KB8NNNC
- R10: Basic (none) -> Y; JLCPCB Part # (none) -> C23186; Manufacturer (none) -> Uniroyal Elec; Manufacturer Part Number (none) -> 0603WAF5101T5E
- R11: footprint Resistor_SMD:R_0603_1608Metric -> Resistor_SMD:R_0805_2012Metric; Basic (none) -> E; JLCPCB Part # (none) -> C17490; Manufacturer (none) -> Uniroyal Elec; Manufacturer Part Number (none) -> 0805W8F1602T5E
- R12: Basic (none) -> Y; JLCPCB Part # (none) -> C21190; Manufacturer (none) -> Uniroyal Elec; Manufacturer Part Number (none) -> 0603WAF1001T5E
- R14: Basic (none) -> Y; JLCPCB Part # (none) -> C4184; Manufacturer (none) -> Uniroyal Elec; Manufacturer Part Number (none) -> 0603WAF2002T5E
- U4: Basic (none) -> X; JLCPCB Part # (none) -> C1855818; Manufacturer (none) -> Texas Instruments; Manufacturer Part Number (none) -> DRV8874PWPR
