File: dc-motor-driver.kicad_sch (KiCad schematic)
At the start: 13 parts, among them U4 DRV8874

Commit message: bom: change dc driver bulk capacitors P#
Parts:
- C11: JLCPCB Part # C2918361 -> C46550411; Manufacturer ROQANG -> jieerrui; Manufacturer Part Number RVT1E221M0607 -> JVJ35V220M6x8
Changed lines of the file:
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@@
 			)
 		)
-		(property "JLCPCB Part #" "C2918361"
+		(property "JLCPCB Part #" "C46550411"
 			(at 180.34 111.76 0)
 			(effects
@@
 			)
 		)
-		(property "Manufacturer" "ROQANG"
+		(property "Manufacturer" "jieerrui"
 			(at 180.34 111.76 0)
 			(effects
@@
 			)
 		)
-		(property "Manufacturer Part Number" "RVT1E221M0607"
+		(property "Manufacturer Part Number" "JVJ35V220M6x8"
 			(at 180.34 111.76 0)
 			(effects
